Commit message: update vehicle fbx file

File: tutorial_vehicle_description/urdf/vehicle.xacro (robot description, xacro)
@@ -8,5 +8,5 @@
       <origin xyz="${vehicle_info['/**']['ros__parameters']['wheel_base']/2.0} 0 0" rpy="${pi/2.0} 0 ${pi}"/>
       <geometry>
-        <mesh filename="package://tutorial_vehicle_description/mesh/vehicle.fbx" scale="1 1 1"/>
+        <mesh filename="package://tutorial_vehicle_description/mesh/tutorial_vehicle.fbx" scale="1 1 1"/>
       </geometry>
     </visual>
